File: PCB/S21/S21.kicad_sch (KiCad schematic)
At the start: 32 parts, among them J1 1x5, J2 Shelly, J3 USB-PROG, J4 1x5, Q1 BSS138PS, Q2 BSS138PS, U2 ESP32-S3-MINI-1, U3 MD8942

Commit message: Render and cases
Parts:
- renumbered C1 to C2, C2 to C5, C3 to C6, D1 to D4, R1 to R3, U2 to U4
Other:
- title: Daikin ESP32-PICO-MINI module -> S21
