File: PCB/ISO7816/ISO7816.kicad_pcb (KiCad board)
At the start: 2 copper layers, 68 x 81 mm, 54 parts, among them J1 Conn_01x02, J3 Conn_01x08, J4 Conn_01x08, J6 USB-C-Socket-H, J7 TC2030-USB-NL-DS, Q1 BSS138PS, Q2 BSS138PS, Q3 BSS138PS, Q4 BSS84, U1 ESP32-S3-MINI-1-N4R2, U2 SN74LVC1T45DCK, U3 TPS562246, U4 TPS22916CNYFPR, U5 TPS22916CNYFPR, U6 SN74LVC1T45DCK

Commit message: Tweak PCB
Parts:
- moved C24 28.5 mm to (201.4, 81.4)
